Commit message: implementation: added deadman switch, added water_world, depth control, buoyancy

File: src/auv_description/urdf/cube/cube.urdf (robot description, URDF)
Before this commit: robot auv, 1 links, 0 joints
Links:
- link cube_link: mass 1.0 -> 1000.0

Commit message: implementations: added camera sensor, modularized/parameterized cube auv, WIP lidar sensor, edited readme

File: src/auv_description/urdf/cube/cube.urdf (robot description, URDF)
Before this commit: robot auv, 1 links, 0 joints
Links:
- added link camera_link, mass 0.1; collision box size=0.1 0.1 0.1; visual box size=0.1 0.1 0.1
- added link camera_optical_frame
- link cube_link: mass 1000.0 -> 999.9
Joints:
- added joint camera_joint: type fixed, parent cube_link, child camera_link, origin xyz=0.55 0 0 rpy=0 0 0
- added joint camera_optical_joint: type fixed, parent camera_link, child camera_optical_frame, origin xyz=0 0 0 rpy=-1.57079632679 0 -1.57079632679
